File: plate/laser_metal_Alps/skean-plate.kicad_pcb (KiCad board)
At the start: 2 copper layers, 153.2 x 95.3 mm, 27 parts, among them K1 KEYSW, K10 KEYSW, K11 KEYSW, K12 KEYSW, K13 KEYSW, K14 KEYSW, K15 KEYSW, K16 KEYSW, K17 KEYSW, K18 KEYSW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

Commit message: Updated laser cutting files
Parts:
- H3, H4, H5, H8, H9: footprint kbd:M2_Hole_TH_mod -> kbd:M2_Hole_Edge_Cut
Routing:
- added copper zone on B.Cu, net (none)
- added copper zone on F.Cu, net (none)
Changed lines of the file:
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@@
     (fp_line (start 9.525 -9.525) (end -9.525 -9.525) (layer "F.Fab") (width 0.15))
   )
-  (footprint "kbd:M2_Hole_TH_mod" (layer "F.Cu")
+  (footprint "kbd:M2_Hole_Edge_Cut" (layer "F.Cu")
     (at 128.721463 40.374367)
     (property "Sheet file" "rt22-plate.kicad_sch")
     (property "Sheet name" "")
-    (fp_text reference "H8" (at 0 0.5) (layer "F.SilkS")
-      (effects (font (size 1 1) (thickness 0.15)))
-    )
-    (fp_text value "MountingHole" (at 0 -0.5) (layer "F.Fab")
-      (effects (font (size 1 1) (thickness 0.15)))
-    )
-    (fp_text user "${REFERENCE}" (at 0.3 0) (layer "F.Fab")
+    (fp_text reference "H8" (at 0 1.9) (layer "Dwgs.User")
+      (effects (font (size 1 1) (thickness 0.15)))
+    )
+    (fp_text value "MountingHole" (at 0 -1.8) (layer "F.Fab")
       (effects (font (size 1 1) (thickness 0.15)))
     )
     (fp_circle (center 0 0) (end 1.15 0) (layer "Edge.Cuts") (width 0.1) (fill none))
-    (pad "" thru_hole circle (at 0 0) (size 4.2 4.2) (drill 2.3) (layers *.Cu *.Mask))
   )
   (footprint "kbd:SW_Hole_ALPS" (layer "F.Cu")
@@
     (fp_line (start -9.525 9.525) (end 9.525 9.525) (layer "F.Fab") (width 0.15))
   )
-  (footprint "kbd:M2_Hole_TH_mod" (layer "F.Cu")
+  (footprint "kbd:M2_Hole_Edge_Cut" (layer "F.Cu")
     (at 71.621463 38.074367)
     (property "Sheet file" "rt22-plate.kicad_sch")
     (property "Sheet name" "")
-    (fp_text reference "H4" (at 0 0.5) (layer "F.SilkS")
-      (effects (font (size 1 1) (thickness 0.15)))
-    )
-    (fp_text value "MountingHole" (at 0 -0.5) (layer "F.Fab")
-      (effects (font (size 1 1) (thickness 0.15)))
-    )
-    (fp_text user "${REFERENCE}" (at 0.3 0) (layer "F.Fab")
+    (fp_text reference "H4" (at 0 1.9) (layer "Dwgs.User")
+      (effects (font (size 1 1) (thickness 0.15)))
+    )
+    (fp_text value "MountingHole" (at 0 -1.8) (layer "F.Fab")
       (effects (font (size 1 1) (thickness 0.15)))
     )
     (fp_circle (center 0 0) (end 1.15 0) (layer "Edge.Cuts") (width 0.1) (fill none))
-    (pad "" thru_hole circle (at 0 0) (size 4.2 4.2) (drill 2.3) (layers *.Cu *.Mask))
   )
   (footprint "kbd:SW_Hole_ALPS" (layer "F.Cu")
@@
     (fp_line (start -9.525 -9.525) (end -9.525 9.525) (layer "F.Fab") (width 0.15))
   )
-  (footprint "kbd:M2_Hole_TH_mod" (layer "F.Cu")
+  (footprint "kbd:M2_Hole_Edge_Cut" (layer "F.Cu")
     (at 33.621463 47.474367)
     (property "Sheet file" "rt22-plate.kicad_sch")
     (property "Sheet name" "")
-    (fp_text reference "H3" (at 0 0.5) (layer "F.SilkS")
-      (effects (font (size 1 1) (thickness 0.15)))
-    )
-    (fp_text value "MountingHole" (at 0 -0.5) (layer "F.Fab")
-      (effects (font (size 1 1) (thickness 0.15)))
-    )
-    (fp_text user "${REFERENCE}" (at 0.3 0) (layer "F.Fab")
+    (fp_text reference "H3" (at 0 1.9) (layer "Dwgs.User")
+      (effects (font (size 1 1) (thickness 0.15)))
+    )
+    (fp_text value "MountingHole" (at 0 -1.8) (layer "F.Fab")
       (effects (font (size 1 1) (thickness 0.15)))
     )
     (fp_circle (center 0 0) (end 1.15 0) (layer "Edge.Cuts") (width 0.1) (fill none))
-    (pad "" thru_hole circle (at 0 0) (size 4.2 4.2) (drill 2.3) (layers *.Cu *.Mask))
   )
   (footprint "kbd:SW_Hole_ALPS" (layer "F.Cu")
@@
     (fp_line (start 9.525 9.525) (end 9.525 -9.525) (layer "F.Fab") (width 0.15))
   )
-  (footprint "kbd:M2_Hole_TH_mod" (layer "F.Cu")
+  (footprint "kbd:M2_Hole_Edge_Cut" (layer "F.Cu")
     (at 71.721463 79.774367)
     (property "Sheet file" "rt22-plate.kicad_sch")
     (property "Sheet name" "")
-    (fp_text reference "H5" (at 0 0.5) (layer "F.SilkS")
-      (effects (font (size 1 1) (thickness 0.15)))
-    )
-    (fp_text value "MountingHole" (at 0 -0.5) (layer "F.Fab")
-      (effects (font (size 1 1) (thickness 0.15)))
-    )
-    (fp_text user "${REFERENCE}" (at 0.3 0) (layer "F.Fab")
+    (fp_text reference "H5" (at 0 1.9) (layer "Dwgs.User")
+      (effects (font (size 1 1) (thickness 0.15)))
+    )
+    (fp_text value "MountingHole" (at 0 -1.8) (layer "F.Fab")
       (effects (font (size 1 1) (thickness 0.15)))
     )
     (fp_circle (center 0 0) (end 1.15 0) (layer "Edge.Cuts") (width 0.1) (fill none))
-    (pad "" thru_hole circle (at 0 0) (size 4.2 4.2) (drill 2.3) (layers *.Cu *.Mask))
   )
   (footprint "kbd:SW_Hole_ALPS" (layer "F.Cu")
@@
     (fp_line (start -9.525 -9.525) (end -9.525 9.525) (layer "F.Fab") (width 0.15))
   )
-  (footprint "kbd:M2_Hole_TH_mod" (layer "F.Cu")
+  (footprint "kbd:M2_Hole_Edge_Cut" (layer "F.Cu")
     (at 142.507505 87.19918)
     (property "Sheet file" "rt22-plate.kicad_sch")
     (property "Sheet name" "")
-    (fp_text reference "H9" (at 0 0.5) (layer "F.SilkS")
-      (effects (font (size 1 1) (thickness 0.15)))
-    )
-    (fp_text value "MountingHole" (at 0 -0.5) (layer "F.Fab")
-      (effects (font (size 1 1) (thickness 0.15)))
-    )
-    (fp_text user "${REFERENCE}" (at 0.3 0) (layer "F.Fab")
+    (fp_text reference "H9" (at 0 1.9) (layer "Dwgs.User")
+      (effects (font (size 1 1) (thickness 0.15)))
+    )
+    (fp_text value "MountingHole" (at 0 -1.8) (layer "F.Fab")
       (effects (font (size 1 1) (thickness 0.15)))
     )
     (fp_circle (center 0 0) (end 1.15 0) (layer "Edge.Cuts") (width 0.1) (fill none))
-    (pad "" thru_hole circle (at 0 0) (size 4.2 4.2) (drill 2.3) (layers *.Cu *.Mask))
   )
   (footprint "kbd:SW_Hole_ALPS" (layer "F.Cu")
@@
   (gr_circle (center 80.721463 28.599368) (end 80.221463 28.599368) (layer "Cmts.User") (width 0.2) (fill none))
   (gr_arc (start 146.221463 21.474368) (mid 146.92857 21.767261) (end 147.221463 22.474368) (layer "Cmts.User") (width 0.2))
-  (gr_circle (center 23.721464 52.349367) (end 23.221464 52.349367) (layer "Cmts.User") (width 0.2) (fill none))
   (gr_line (start 110.221463 19.099367) (end 127.221463 19.099367) (layer "Cmts.User") (width 0.2))
   (gr_circle (center 33.621463 47.474367) (end 32.621463 47.474367) (layer "Cmts.User") (width 0.2) (fill none))
@@
   (gr_arc (start 154.028536 109.150633) (mid 153.42133 109.616559) (end 152.662511 109.516658) (layer "Edge.Cuts") (width 0.2))
   (gr_line (start 34.221464 28.599368) (end 51.221463 28.599368) (layer "Edge.Cuts") (width 0.2))
+  (zone (net 0) (net_name "") (layers F&B.Cu) (hatch edge 0.508)
+    (priority 1)
+    (connect_pads (clearance 0.2))
+    (min_thickness 0.25) (filled_areas_thickness no)
+    (fill yes (mode hatch) (thermal_gap 0.5) (thermal_bridge_width 0.5)
+      (hatch_thickness 0.5) (hatch_gap 0.8) (hatch_orientation 45)
+      (hatch_border_algorithm hatch_thickness) (hatch_min_hole_area 0.3))
+    (polygon
+      (pts
+        (xy 109.221463 19.104952)
+        (xy 128.221463 19.104952)
+        (xy 128.221463 21.504952)
+        (xy 147.221463 21.504952)
+        (xy 147.221463 23.804952)
+        (xy 147.721464 73.349367)
+        (xy 167.821463 85.204952)
+        (xy 153.421463 109.904952)
+        (xy 137.021463 100.504952)
+        (xy 99.721463 95.504952)
+        (xy 90.121463 85.504952)
+        (xy 33.221463 85.604952)
+        (xy 33.221463 61.804952)
+        (xy 14.121463 61.804952)
+        (xy 14.221463 42.904952)
+        (xy 33.221463 42.804952)
+        (xy 33.221463 28.504952)
+        (xy 52.221463 28.504952)
+        (xy 52.221463 26.204952)
+        (xy 71.221463 26.204952)
+        (xy 71.221463 19.004952)
+        (xy 90.221463 19.004952)
+        (xy 90.221463 14.304952)
+        (xy 109.221463 14.304952)
+      )
+    )
+  )
 )
