File: bottom/laser_6col/skean-bottom.kicad_pcb (KiCad board)
At the start: 2 copper layers, 153.2 x 95.3 mm, 5 parts

Commit message: Updated laser cutting files
Parts:
- removed H3: MountingHole, kbd:M2_Hole_TH_mod
- H4, H5, H8, H9: footprint kbd:M2_Hole_TH_mod -> kbd:M2_Hole_Edge_Cut
Other:
- board size 153.2 x 95.3 mm -> 134.2 x 95.3 mm

Commit message: New bottom files for extreme 301230 configurations
Parts:
- added H2: MountingHole, kbd:M2_Hole_Edge_Cut, F.Cu at (51.8, 66.6)
- added H3: MountingHole, kbd:M2_Hole_Edge_Cut, F.Cu at (51.7, 47.6)
Changed lines of the file:
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@@
+  )
+  (footprint "kbd:M2_Hole_Edge_Cut" (layer "F.Cu")
+    (at 51.721463 47.574367)
+    (property "Sheetfile" "skean-bottom.kicad_sch")
+    (property "Sheetname" "")
+    (fp_text reference "H3" (at 0 1.9) (layer "Dwgs.User")
+      (effects (font (size 1 1) (thickness 0.15)))
+    )
+    (fp_text value "MountingHole" (at 0 -1.8) (layer "F.Fab")
+      (effects (font (size 1 1) (thickness 0.15)))
+    )
+    (fp_circle (center 0 0) (end 1.15 0) (layer "Edge.Cuts") (width 0.1) (fill none))
   )
   (footprint "kbd:M2_Hole_Edge_Cut" (layer "F.Cu")
@@
       (effects (font (size 1 1) (thickness 0.15)))
     )
+    (fp_text value "MountingHole" (at 0 -1.8) (layer "F.Fab")
+      (effects (font (size 1 1) (thickness 0.15)))
+    )
+    (fp_circle (center 0 0) (end 1.15 0) (layer "Edge.Cuts") (width 0.1) (fill none))
+  )
+  (footprint "kbd:M2_Hole_Edge_Cut" (layer "F.Cu")
+    (at 51.821463 66.574367)
+    (property "Sheetfile" "skean-bottom.kicad_sch")
+    (property "Sheetname" "")
+    (fp_text reference "H2" (at 0 1.9) (layer "Dwgs.User")
+      (effects (font (size 1 1) (thickness 0.15)))
+    )
