File: pcb/6col/skean.kicad_sch (KiCad schematic)
At the start: 77 parts, among them J2 SWD, J3 USB-C Conn, J4 Conn_01x02_Female, K1 KEYSW, K10 KEYSW, K11 KEYSW, K12 KEYSW, K13 KEYSW, K14 KEYSW, K15 KEYSW, K16 KEYSW, K17 KEYSW, K18 KEYSW, K2 KEYSW, K20 KEYSW, K21 KEYSW, K22 KEYSW, K3 KEYSW, K4 KEYSW, K5 KEYSW, K6 KEYSW, K7 KEYSW, K8 KEYSW, K9 KEYSW, Q2 AO3407, SW1 SW_SPDT, U1 E73-2G4M08S1E, U2 XC6220B331MR-G, U3 TP4054, U4 USBLC6-2SC6, X1 32.768kHz

Commit message: V0.3 solder PCBs
Parts:
- added H0: MountingHole, kbd:M2-MountingHole-Standoff, symbol Mechanical:MountingHole
- J3: footprint kbd:USB-C_C168688_REV -> kbd:USB-C_C168688_REV_V2
- K1, K10, K11, K12, K13, K14, K15, K16, K17, K2, K20, K21, K3, K4, K5, K6, K7, K8, K9: footprint kbd:MX-Alps-1U-REV -> kbd:MX-Alps-Omron-SKCC-Hitek-Futaba-MA-1U-REV
- K18: footprint kbd:MX-Alps-1U-REV -> kbd:MX-Alps-Omron-SKCC-Inv-Hitek-Futaba-MA-1U-REV
- K22: footprint kbd:MX-Alps-1.5U-REV -> kbd:MX-Alps-Omron-SKCC-Hitek-Futaba-MA-1.5U-REV
Connections:
- net PROG: no longer names the net of U1.15 (P0.05/AIN3)
- no-connect marks 6 -> 7
